File: PCB/pico_node/pico_node.kicad_pcb (KiCad board)
At the start: 2 copper layers, 19 parts, among them J1 INMP441, J2 NEO-6M, J3 MD-CD42, J4 RESET_POWER_SW, J5 UART0_DEBUG, J6 UART1_DEBUG, J7 BATTERY, J8 BUCK_5V, Q1 BC547, U1 NRF24L01_Breakout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

Commit message: updated PCB
Parts:
- Q1: footprint Package_TO_SOT_THT:TO-92_Inline -> Package_TO_SOT_THT:TO-92_Inline_Wide
- moved R4 97.4 mm to (148.4, 81.1), turned to 180 degrees
- moved R1 67.1 mm to (176.0, 85.2)
- moved D2 66.6 mm to (147.7, 86.2), turned to 180 degrees
- moved R2 57.4 mm to (190.0, 75.0), turned to -90 degrees
- moved D1 56.1 mm to (196.0, 67.2), turned to 180 degrees
- moved R3 54.7 mm to (200.4, 67.4), turned to -90 degrees
- moved Q1 48.8 mm to (194.3, 72.5), turned to -90 degrees
- moved J4 40.6 mm to (188.4, 64.9), turned to 180 degrees
- moved C1 37.3 mm to (118.7, 59.8), turned to -90 degrees
- moved J2 31.2 mm to (134.7, 72.1)
- moved U1 30.8 mm to (136.3, 54.4)
- moved J6 22.4 mm to (144.7, 64.9)
- moved J5 22.0 mm to (144.7, 39.5)
- moved U2 18.9 mm to (111.0, 57.9)
- moved J8 12.4 mm to (193.2, 49.7)
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Connections:
- J4 pad 1: /RUN -> GND
- J4 pad 2: GND -> /RUN
- J5 pad 1: /GP1 -> /GP0
- J5 pad 2: /GP2 -> /GP1
- R1 pad 1: /GP15 -> /GP17
- R4 pad 1: /GP22 -> /GP13
Routing:
- net /GP7: track 0.00 -> 51.7 mm, vias 0 -> 2
- net /GP5: track 0.00 -> 44.9 mm, vias 0 -> 2
- net +3.3V: track 0.00 -> 44.7 mm, vias 0 -> 2
- net /GP3: track 0.00 -> 35.9 mm
- net /GP2: track 0.00 -> 26.4 mm, vias 0 -> 2
- net /GP8: track 0.00 -> 24.5 mm
- net /GP9: track 0.00 -> 24.5 mm
- net /GP18: track 0.00 -> 22.1 mm, vias 0 -> 2
- net /GP6: track 0.00 -> 20.9 mm
- net /GP4: track 0.00 -> 18.5 mm
- net Net-(Q1-B): track 0.00 -> 16.1 mm
- net VBUS: track 0.00 -> 15.6 mm
- net /RUN: track 0.00 -> 15.5 mm
- net Net-(C1-+): track 0.00 -> 13.0 mm, vias 0 -> 2
- net Net-(R4--): track 0.00 -> 9.98 mm
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Other:
- board outline added: 107.3 x 53.3 mm
