File: PCB/pico_node/pico_node.kicad_sch (KiCad schematic)
At the start: 19 parts, among them J1 INMP441, J2 NEO-6M, J3 MD-CD42, J4 RESET_POWER_SW, J5 UART0_DEBUG, J6 UART1_DEBUG, J7 BATTERY, J8 BUCK_5V, Q1 BC547, U1 NRF24L01_Breakout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

Commit message: updated PCB
Parts:
- Q1: footprint Package_TO_SOT_THT:TO-92_Inline -> Package_TO_SOT_THT:TO-92_Inline_Wide
Connections:
- net GND: now also J4.1 (Pin_1); no longer J4.2 (Pin_2)
- net GP0: now also J5.1 (Pin_1)
- net GP1: now also J5.2 (Pin_2); no longer J5.1 (Pin_1)
- net GP13: now also R4.1 (+)
- net GP15: no longer R1.1 (+)
- net GP17: now also R1.1 (+)
- net GP2: no longer J5.2 (Pin_2)
- net GP22: no longer R4.1 (+)
- net RUN: now also J4.2 (Pin_2); no longer J4.1 (Pin_1)
Changed lines of the file:
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@@
 	(wire
 		(pts
-			(xy 55.88 33.02) (xy 62.23 33.02)
+			(xy 50.165 161.925) (xy 50.165 160.02)
 		)
 		(stroke
@@
 	(wire
 		(pts
-			(xy 50.165 161.925) (xy 50.165 160.02)
+			(xy 180.34 84.455) (xy 167.005 84.455)
 		)
 		(stroke
@@
 	(wire
 		(pts
-			(xy 180.34 84.455) (xy 167.005 84.455)
+			(xy 60.325 62.23) (xy 72.39 62.23)
 		)
 		(stroke
@@
 	(wire
 		(pts
-			(xy 60.325 62.23) (xy 72.39 62.23)
+			(xy 55.88 35.56) (xy 62.23 35.56)
 		)
 		(stroke
@@
 	(wire
 		(pts
-			(xy 54.61 35.56) (xy 62.23 35.56)
+			(xy 180.34 95.885) (xy 167.005 95.885)
 		)
 		(stroke
@@
 	(wire
 		(pts
-			(xy 180.34 95.885) (xy 167.005 95.885)
+			(xy 54.61 33.02) (xy 62.23 33.02)
 		)
 		(stroke
@@
 		)
 	)
-	(label "GP1"
+	(label "GP0"
 		(at 65.405 103.505 0)
 		(effects
@@
 		)
 	)
-	(label "GP22"
+	(label "GP13"
 		(at 210.185 120.65 0)
 		(effects
@@
 		)
 	)
-	(label "GP15"
+	(label "GP17"
 		(at 218.44 75.565 0)
 		(effects
@@
 		)
 	)
-	(label "GP2"
+	(label "GP1"
 		(at 65.405 106.045 0)
 		(effects
@@
 	)
 	(label "RUN"
-		(at 55.88 33.02 0)
+		(at 55.88 35.56 0)
 		(effects
 			(font
@@
 	(symbol
 		(lib_id "power:GND")
-		(at 54.61 35.56 270)
+		(at 54.61 33.02 270)
 		(unit 1)
 		(exclude_from_sim no)
@@
 		(fields_autoplaced yes)
 		(property "Reference" "#PWR022"
-			(at 48.26 35.56 0)
+			(at 48.26 33.02 0)
 			(effects
 				(font
@@
 		)
 		(property "Value" "GND"
-			(at 50.8 35.5599 90)
+			(at 50.8 33.0199 90)
 			(effects
 				(font
@@
 		)
 		(property "Footprint" ""
-			(at 54.61 35.56 0)
+			(at 54.61 33.02 0)
 			(effects
 				(font
@@
 		)
 		(property "Datasheet" ""
-			(at 54.61 35.56 0)
+			(at 54.61 33.02 0)
 			(effects
 				(font
@@
 		)
 		(property "Description" "Power symbol creates a global label with name \"GND\" , ground"
-			(at 54.61 35.56 0)
+			(at 54.61 33.02 0)
 			(effects
 				(font
@@
 			)
 		)
-		(property "Footprint" "Package_TO_SOT_THT:TO-92_Inline"
+		(property "Footprint" "Package_TO_SOT_THT:TO-92_Inline_Wide"
 			(at 254 77.47 0)
 			(effects
