File: PCB/pico_node/pico_node.kicad_sch (KiCad schematic)
At the start: 19 parts, among them J1 INMP441, J2 NEO-6M, J3 MD-CD42, J4 RESET_POWER_SW, J5 UART0_DEBUG, J6 UART1_DEBUG, J7 BATTERY, J8 BUCK_5V, Q1 BC547, U1 NRF24L01_Breakout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

Commit message: Update on pico_node pcb
Parts:
- R3: footprint Resistor_THT:R_Axial_DIN0207_L6.3mm_D2.5mm_P10.16mm_Horizontal -> Resistor_SMD:R_1210_3225Metric_Pad1.30x2.65mm_HandSolder
Changed lines of the file:
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@@
 			)
 		)
-		(property "Footprint" "Resistor_THT:R_Axial_DIN0207_L6.3mm_D2.5mm_P10.16mm_Horizontal"
+		(property "Footprint" "Resistor_SMD:R_1210_3225Metric_Pad1.30x2.65mm_HandSolder"
 			(at 251.46 63.5 0)
 			(effects
